File: PCB/RS485-Gassensor/output.kicad_sch (KiCad schematic)
At the start: 24 parts, among them J6 Conn_01x02_Pin, J7 Conn_01x02_Pin, U6 AD8676, U7 LT1785xS8, U9 AD8676

Commit message: made For NAP505 and NAP550
Parts:
- added J10: Conn_01x02, Connector_PinHeader_2.54mm:PinHeader_1x02_P2.54mm_Vertical, symbol Connector_Generic:Conn_01x02
- added R10 (x2): R10K, Resistor_SMD:R_0603_1608Metric, symbol Device:R
Connections:
- net +3.3V: now also R10.1, R10.2
- new net I2C_SCL: R10.2
- new net I2C_SDA: R10.1
Changed lines of the file:
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@@
   (junction (at 210.82 116.84) (diameter 0) (color 0 0 0 0)
   )
+  (junction (at 44.45 129.54) (diameter 0) (color 0 0 0 0)
+  )
   (junction (at 191.77 127) (diameter 0) (color 0 0 0 0)
   )
@@
   (junction (at 121.92 52.07) (diameter 0) (color 0 0 0 0)
   )
+  (junction (at 49.53 127) (diameter 0) (color 0 0 0 0)
+  )
   (junction (at 168.91 105.41) (diameter 0) (color 0 0 0 0)
   )
@@
     (stroke (width 0) (type default))
   )
+  (wire (pts (xy 44.45 129.54) (xy 44.45 132.08))
+    (stroke (width 0) (type default))
+  )
   (wire (pts (xy 168.91 101.6) (xy 168.91 105.41))
     (stroke (width 0) (type default))
@@
     (stroke (width 0) (type default))
   )
+  (wire (pts (xy 44.45 132.08) (xy 35.56 132.08))
+    (stroke (width 0) (type default))
+  )
   (wire (pts (xy 193.04 63.5) (xy 190.5 63.5))
     (stroke (width 0) (type default))
@@
     (stroke (width 0) (type default))
   )
+  (wire (pts (xy 44.45 120.65) (xy 44.45 129.54))
+    (stroke (width 0) (type default))
+  )
   (wire (pts (xy 168.91 139.7) (xy 168.91 142.24))
     (stroke (width 0) (type default))
@@
     (stroke (width 0) (type default))
   )
+  (wire (pts (xy 49.53 127) (xy 57.15 127))
+    (stroke (width 0) (type default))
+  )
   (wire (pts (xy 210.82 138.43) (xy 210.82 116.84))
     (stroke (width 0) (type default))
@@
     (stroke (width 0) (type default))
   )
+  (wire (pts (xy 44.45 129.54) (xy 57.15 129.54))
+    (stroke (width 0) (type default))
+  )
   (wire (pts (xy 193.04 63.5) (xy 193.04 64.77))
     (stroke (width 0) (type default))
@@
     (stroke (width 0) (type default))
   )
+  (wire (pts (xy 49.53 120.65) (xy 49.53 127))
+    (stroke (width 0) (type default))
+  )
   (wire (pts (xy 128.27 128.27) (xy 128.27 124.46))
     (stroke (width 0) (type default))
@@
     (stroke (width 0) (type default))
   )
+  (wire (pts (xy 49.53 111.76) (xy 49.53 113.03))
+    (stroke (width 0) (type default))
+  )
+  (wire (pts (xy 35.56 124.46) (xy 40.64 124.46))
+    (stroke (width 0) (type default))
+  )
   (wire (pts (xy 180.34 127) (xy 180.34 121.92))
     (stroke (width 0) (type default))
@@
     (stroke (width 0) (type default))
   )
+  (wire (pts (xy 44.45 111.76) (xy 44.45 113.03))
+    (stroke (width 0) (type default))
+  )
   (wire (pts (xy 172.72 73.66) (xy 172.72 66.04))
     (stroke (width 0) (type default))
@@
     (stroke (width 0) (type default))
   )
+  (wire (pts (xy 40.64 124.46) (xy 40.64 127))
+    (stroke (width 0) (type default))
+  )
   (wire (pts (xy 193.04 39.37) (xy 193.04 40.64))
     (stroke (width 0) (type default))
@@
   )
   (wire (pts (xy 154.94 27.94) (xy 162.56 27.94))
+    (stroke (width 0) (type default))
+  )
+  (wire (pts (xy 40.64 127) (xy 49.53 127))
     (stroke (width 0) (type default))
   )
@@
     )
   )
+  (global_label "I2C_SDA" (shape input) (at 35.56 132.08 180) (fields_autoplaced)
+    (effects (font (size 1.27 1.27)) (justify right))
+    (property "Intersheetrefs" "${INTERSHEET_REFS}" (at 25.0342 132.08 0)
+      (effects (font (size 1.27 1.27)) (justify right) hide)
+    )
+  )
   (global_label "UART_TX" (shape input) (at 152.4 129.54 180) (fields_autoplaced)
     (effects (font (size 1.27 1.27)) (justify right))
@@
     )
   )
+  (global_label "I2C_SCL" (shape input) (at 35.56 124.46 180) (fields_autoplaced)
+    (effects (font (size 1.27 1.27)) (justify right))
+    (property "Intersheetrefs" "${INTERSHEET_REFS}" (at 25.0947 124.46 0)
+      (effects (font (size 1.27 1.27)) (justify right) hide)
+    )
+  )
   (global_label "analog_PWM_NO" (shape input) (at 142.24 60.96 180) (fields_autoplaced)
     (effects (font (size 1.27 1.27)) (justify right))
@@
         (path "/3e460a3b-bdfc-40e9-ad81-ef9b20842c44/9d83f588-fa0e-41f8-8cf7-9ca24a12f734"
           (reference "#PWR035") (unit 1)
+        )
+      )
+    )
+  )
+  (symbol (lib_id "power:+3.3V") (at 49.53 111.76 0) (unit 1)
+    (in_bom yes) (on_board yes) (dnp no)
+    (property "Reference" "#PWR034" (at 49.53 115.57 0)
+      (effects (font (size 1.27 1.27)) hide)
+    )
+    (property "Value" "+3.3V" (at 54.61 110.49 0)
+      (effects (font (size 1.27 1.27)))
+    )
+    (property "Footprint" "" (at 49.53 111.76 0)
+      (effects (font (size 1.27 1.27)) hide)
+    )
+    (property "Datasheet" "" (at 49.53 111.76 0)
+      (effects (font (size 1.27 1.27)) hide)
+    )
+    (pin "1")
+    (instances
+      (project "RS485-Gassensor"
+        (path "/3e460a3b-bdfc-40e9-ad81-ef9b20842c44"
+          (reference "#PWR034") (unit 1)
+        )
+        (path "/3e460a3b-bdfc-40e9-ad81-ef9b20842c44/9d83f588-fa0e-41f8-8cf7-9ca24a12f734"
+          (reference "#PWR055") (unit 1)
         )
       )
@@
     )
   )
+  (symbol (lib_id "Device:R") (at 49.53 116.84 0) (unit 1)
+    (in_bom yes) (on_board yes) (dnp no)
+    (property "Reference" "R10" (at 52.07 115.57 0)
+      (effects (font (size 1.27 1.27)) (justify left))
+    )
+    (property "Value" "R10K" (at 52.07 118.11 0)
+      (effects (font (size 1.27 1.27)) (justify left))
+    )
+    (property "Footprint" "Resistor_SMD:R_0603_1608Metric" (at 47.752 116.84 90)
+      (effects (font (size 1.27 1.27)) hide)
+    )
+    (property "Datasheet" "~" (at 49.53 116.84 0)
+      (effects (font (size 1.27 1.27)) hide)
+    )
+    (pin "1")
+    (pin "2")
+    (instances
+      (project "RS485-Gassensor"
+        (path "/3e460a3b-bdfc-40e9-ad81-ef9b20842c44"
+          (reference "R10") (unit 1)
+        )
+        (path "/3e460a3b-bdfc-40e9-ad81-ef9b20842c44/9d83f588-fa0e-41f8-8cf7-9ca24a12f734"
+          (reference "R31") (unit 1)
+        )
+      )
+    )
+  )
   (symbol (lib_id "Device:R") (at 193.04 78.74 0) (unit 1)
     (in_bom yes) (on_board yes) (dnp no) (fields_autoplaced)
@@
     )
   )
+  (symbol (lib_id "Device:R") (at 44.45 116.84 180) (unit 1)
+    (in_bom yes) (on_board yes) (dnp no)
+    (property "Reference" "R10" (at 41.91 118.11 0)
+      (effects (font (size 1.27 1.27)) (justify left))
+    )
+    (property "Value" "R10K" (at 41.91 115.57 0)
+      (effects (font (size 1.27 1.27)) (justify left))
+    )
+    (property "Footprint" "Resistor_SMD:R_0603_1608Metric" (at 46.228 116.84 90)
+      (effects (font (size 1.27 1.27)) hide)
+    )
+    (property "Datasheet" "~" (at 44.45 116.84 0)
+      (effects (font (size 1.27 1.27)) hide)
+    )
+    (pin "1")
+    (pin "2")
+    (instances
+      (project "RS485-Gassensor"
+        (path "/3e460a3b-bdfc-40e9-ad81-ef9b20842c44"
+          (reference "R10") (unit 1)
+        )
+        (path "/3e460a3b-bdfc-40e9-ad81-ef9b20842c44/9d83f588-fa0e-41f8-8cf7-9ca24a12f734"
+          (reference "R30") (unit 1)
+        )
+      )
+    )
+  )
   (symbol (lib_id "Device:R") (at 151.13 60.96 90) (unit 1)
     (in_bom yes) (on_board yes) (dnp no)
@@
         (path "/3e460a3b-bdfc-40e9-ad81-ef9b20842c44/9d83f588-fa0e-41f8-8cf7-9ca24a12f734"
           (reference "R17") (unit 1)
+        )
+      )
+    )
+  )
+  (symbol (lib_id "Connector_Generic:Conn_01x02") (at 62.23 127 0) (unit 1)
+    (in_bom yes) (on_board yes) (dnp no) (fields_autoplaced)
+    (property "Reference" "J10" (at 64.77 127 0)
+      (effects (font (size 1.27 1.27)) (justify left))
+    )
+    (property "Value" "Conn_01x02" (at 64.77 129.54 0)
+      (effects (font (size 1.27 1.27)) (justify left))
+    )
+    (property "Footprint" "Connector_PinHeader_2.54mm:PinHeader_1x02_P2.54mm_Vertical" (at 62.23 127 0)
+      (effects (font (size 1.27 1.27)) hide)
+    )
+    (property "Datasheet" "~" (at 62.23 127 0)
+      (effects (font (size 1.27 1.27)) hide)
+    )
+    (pin "1")
+    (pin "2")
+    (instances
+      (project "RS485-Gassensor"
+        (path "/3e460a3b-bdfc-40e9-ad81-ef9b20842c44/9d83f588-fa0e-41f8-8cf7-9ca24a12f734"
+          (reference "J10") (unit 1)
         )
       )
@@
         )
       )
+    )
+  )
+  (symbol (lib_id "power:+3.3V") (at 44.45 111.76 0) (unit 1)
+    (in_bom yes) (on_board yes) (dnp no)
+    (property "Reference" "#PWR034" (at 44.45 115.57 0)
+      (effects (font (size 1.27 1.27)) hide)
+    )
+    (property "Value" "+3.3V" (at 39.37 110.49 0)
+      (effects (font (size 1.27 1.27)))
+    )
+    (property "Footprint" "" (at 44.45 111.76 0)
+      (effects (font (size 1.27 1.27)) hide)
+    )
+    (property "Datasheet" "" (at 44.45 111.76 0)
+      (effects (font (size 1.27 1.27)) hide)
+    )
+    (pin "1")
+    (instances
+      (project "RS485-Gassensor"
+        (path "/3e460a3b-bdfc-40e9-ad81-ef9b20842c44"
+          (reference "#PWR034") (unit 1)
+        )
+        (path "/3e460a3b-bdfc-40e9-ad81-ef9b20842c44/9d83f588-fa0e-41f8-8cf7-9ca24a12f734"
+          (reference "#PWR054") (unit 1)
+        )
+      )

Commit message: code and hardware imrovement V2
added I2C, and modbus functionailties
Connections:
- net I2C_SCL: now also J10.1 (Pin_1)
- net I2C_SDA: now also J10.2 (Pin_2)
